Commit message: nailed it

File: pendulum.urdf (robot description, URDF)
Before this commit: robot pendulum, 4 links, 3 joints
Links:
- link link_1: geometry visual cylinder length=0.8 radius=0.01
Joints:
- joint joint_1: origin xyz=0.0 0 0 rpy=0 3.1415 0 -> xyz=0.0 0 0 rpy=0 3.14159265359 0
- joint joint_eef: origin xyz=0 0 1.2 rpy=0 0 0 -> xyz=0 0 0.8 rpy=0 0 0

Commit message: Uncommit

File: pendulum.urdf (robot description, URDF)
Before this commit: robot pendulum, 4 links, 3 joints
Links:
- link link_1: geometry visual cylinder length=1.2 radius=0.01
Joints:
- joint joint_1: origin xyz=0.0 0 0 rpy=0 3.14159265359 0 -> xyz=0.0 0 0 rpy=0 3.1415 0
- joint joint_eef: origin xyz=0 0 0.8 rpy=0 0 0 -> xyz=0 0 1.2 rpy=0 0 0
